Commit message: add camera

File: robots/robot.urdf (robot description, URDF)
Before this commit: robot onshape, 7 links, 6 joints
Links:
- added link camera_link
- added link camera_link_optical
Joints:
- added joint camera_joint: type fixed, parent shoulder_5, child camera_link, origin xyz=0 0.059 0.019 rpy=3.1415926535897931 0 1.57079632679, axis 0 0 0
- added joint camera_optical_joint: type fixed, parent camera_link, child camera_link_optical, origin xyz=0 0 0 rpy=-1.57079632679 0 -1.57079632679
